File: l289/L298.brd (EAGLE design)
At the start: 160 x 100 mm, 22 parts, among them IC1 L298, IC3 7805TV

Commit message: second version
Parts:
- removed JP1, JP2: (no value), pinhead:1X05
- added JP4: (no value), pinhead:2X06
- added JP5: (no value), pinhead:1X03
- JP3: device pinhead:2X05 -> pinhead:1X03
- moved R1 203.5 mm to (104.1, 66.7), turned to 270 degrees
- moved LED1 198.5 mm to (99.1, 67.3), turned to 180 degrees
- moved JP3 198.0 mm to (72.4, 80.0), turned to 180 degrees
- moved D9 188.7 mm to (95.2, 81.3), turned to 270 degrees
- moved D8 181.0 mm to (92.1, 81.3), turned to 270 degrees
- moved D6 175.0 mm to (98.4, 81.3), turned to 90 degrees
- moved D5 172.6 mm to (101.6, 81.3), turned to 90 degrees
- moved D7 157.5 mm to (56.5, 87.6), turned to 270 degrees
- moved MOTOR2 143.7 mm to (113.0, 90.2), turned to 270 degrees
- moved D4 141.3 mm to (59.7, 87.6), turned to 90 degrees
- moved J1 138.6 mm to (106.0, 53.3), turned to 90 degrees
- moved D3 131.4 mm to (53.3, 87.6), turned to 270 degrees
- moved IC1 128.7 mm to (76.2, 94.6)
- moved MOTOR1 126.2 mm to (81.3, 68.6), turned to 180 degrees
- moved D2 123.6 mm to (50.2, 87.6), turned to 90 degrees
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Connections:
- new net VSS: C2.1, D1.C, D2.C, D4.C, D5.C, D6.C, IC1.4, IC3.1, R1.2
- net +12V: no longer C2.1, D2.C, D4.C, D5.C, D6.C, IC1.4, IC3.1, R1.2
- net +5V: now also JP4.1, JP4.11, JP4.3, JP4.5, JP4.7, JP4.9; no longer JP1.5, JP2.5, JP3.1, JP3.3, JP3.5, JP3.7, JP3.9
- net ENA: now also JP3.2; no longer JP1.4
- net ENB: now also JP5.2; no longer JP2.4
- net GND: now also JP4.10, JP4.12, JP4.2, JP4.4, JP4.6, JP4.8; no longer D1.C, JP1.1, JP2.1, JP3.10, JP3.2, JP3.4, JP3.6, JP3.8
- net IN1: now also JP3.3; no longer JP1.3
- net IN2: now also JP3.1; no longer JP1.2
- net IN3: now also JP5.3; no longer JP2.3
- net IN4: now also JP5.1; no longer JP2.2
