File: l289/L298.brd (EAGLE design)
At the start: 160 x 100 mm, 22 parts, among them IC1 L298, IC3 7805TV

Commit message: Added frame in SCH
Parts:
- moved C3 2.29 mm to (75.6, 73.7), turned to 90 degrees
Changed lines of the file:
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@@
 <element name="C1" library="resistor" package="C050-024X044" value="1uF" x="103.505" y="58.42" rot="R180"/>
 <element name="C2" library="resistor" package="C050-024X044" value="0.33uF" x="68.58" y="73.66"/>
-<element name="C3" library="resistor" package="C050-024X044" value="0.1uF" x="77.47" y="74.93"/>
+<element name="C3" library="resistor" package="C050-024X044" value="0.1uF" x="75.565" y="73.66" rot="R90"/>
 <element name="D1" library="adafruit" package="DO41-10" value="1N4004" x="74.295" y="64.77"/>
 <element name="IC1" library="st-microelectronics" package="MULTIWATT-15" value="L298" x="76.2" y="94.615">
@@
 <wire x1="88.265" y1="76.835" x2="88.265" y2="69.85" width="0" layer="19" extent="1-1"/>
 <wire x1="92.075" y1="81.915" x2="88.265" y2="76.835" width="0" layer="19" extent="1-1"/>
-<wire x1="80.01" y1="74.93" x2="88.265" y2="76.835" width="0" layer="19" extent="1-1"/>
-<wire x1="71.12" y1="73.66" x2="80.01" y2="74.93" width="0" layer="19" extent="1-1"/>
+<wire x1="75.565" y1="76.2" x2="88.265" y2="76.835" width="0" layer="19" extent="1-1"/>
+<wire x1="71.12" y1="73.66" x2="75.565" y2="76.2" width="0" layer="19" extent="1-1"/>
 <wire x1="60.325" y1="82.55" x2="71.12" y2="73.66" width="0" layer="19" extent="1-1"/>
 <wire x1="57.15" y1="76.835" x2="60.325" y2="82.55" width="0" layer="19" extent="1-1"/>
-<wire x1="76.2" y1="92.075" x2="80.01" y2="74.93" width="0" layer="19" extent="1-1"/>
+<wire x1="76.2" y1="92.075" x2="75.565" y2="76.2" width="0" layer="19" extent="1-1"/>
 </signal>
 <signal name="+12V">
@@
 <wire x1="111.76" y1="63.5" x2="111.76" y2="66.04" width="0" layer="19" extent="1-1"/>
 <wire x1="90.805" y1="69.85" x2="111.76" y2="71.12" width="0" layer="19" extent="1-1"/>
-<wire x1="74.93" y1="74.93" x2="90.805" y2="69.85" width="0" layer="19" extent="1-1"/>
-<wire x1="77.47" y1="86.995" x2="74.93" y2="74.93" width="0" layer="19" extent="1-1"/>
+<wire x1="75.565" y1="71.12" x2="90.805" y2="69.85" width="0" layer="19" extent="1-1"/>
+<wire x1="77.47" y1="86.995" x2="75.565" y2="71.12" width="0" layer="19" extent="1-1"/>
 </signal>
 <signal name="N$1">

Commit message: Routed halfway through
Parts:
- removed J1: (no value), SparkFun-Connectors:JST-2-PTH-NS
- added X3: (no value), con-wago-500:W237-102
- moved C2 23.6 mm to (57.8, 52.7), turned to 180 degrees
- moved X2 12.1 mm to (108.6, 89.5)
- moved C3 8.28 mm to (76.2, 81.9)
- moved D4 7.62 mm to (56.5, 81.9)
- moved D7 6.99 mm to (64.1, 81.9)
- moved D1 5.46 mm to (69.8, 61.6), turned to 180 degrees
- moved IC3 3.86 mm to (88.9, 68.6), turned to 180 degrees
- moved JP3 3.18 mm to (72.4, 76.8)
- moved JP5 3.18 mm to (80.0, 76.8)
Connections:
- net +12V: now also X3.1; no longer J1.2
- net GND: now also X3.2; no longer J1.1
Routing:
- net N$3: track 0.00 -> 30.9 mm
- net N$2: track 0.00 -> 29.6 mm
- net GND: track 0.00 -> 24.2 mm
- net N$4: track 0.00 -> 23.5 mm
- net N$1: track 0.00 -> 23.1 mm
- net VSS: track 0.00 -> 16.6 mm
- net ENA: track 0.00 -> 15.8 mm
- net IN4: track 0.00 -> 15.8 mm
- net IN3: track 0.00 -> 15.8 mm
- net +5V: track 0.00 -> 14.2 mm
- net IN1: track 0.00 -> 11.2 mm
- net IN2: track 0.00 -> 10.2 mm
- net ENB: track 0.00 -> 10.2 mm
