File: l289/L298.sch (EAGLE design)
At the start: 22 parts, among them IC1 L298, IC3 7805TV

Commit message: Routed halfway through
Parts:
- removed J1: (no value), SparkFun-Connectors:M02-JST-2-PTH-NO_SILK
- added X3: (no value), con-wago-500:W237-102
Connections:
- net +12V: now also X3-1.KL; no longer J1.2
- net GND: now also X3-2.KL; no longer J1.1
Other:
- moved on the sheet: C1, D1, JP3
Changed lines of the file:
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@@
 <parts>
 <part name="IC1" library="st-microelectronics" deviceset="L298" device=""/>
-<part name="J1" library="SparkFun-Connectors" deviceset="M02" device="-JST-2-PTH-NO_SILK"/>
 <part name="SUPPLY1" library="supply2" deviceset="+12V" device=""/>
 <part name="SUPPLY2" library="supply2" deviceset="GND" device=""/>
@@
 <part name="X2" library="con-wago-500" deviceset="W237-102" device=""/>
 <part name="U$1" library="CustomLib" deviceset="FRAME_A4_ADAFRUIT" device=""/>
+<part name="X3" library="con-wago-500" deviceset="W237-102" device=""/>
 </parts>
 <sheets>
@@
 <instances>
 <instance part="IC1" gate="L298" x="66.04" y="53.34"/>
-<instance part="J1" gate="G$1" x="-5.08" y="73.66"/>
-<instance part="SUPPLY1" gate="+12V" x="7.62" y="83.82"/>
-<instance part="SUPPLY2" gate="GND" x="7.62" y="66.04"/>
-<instance part="C1" gate="G$1" x="15.24" y="76.2"/>
-<instance part="SUPPLY3" gate="+12V" x="15.24" y="93.98" rot="R90"/>
-<instance part="D1" gate="1" x="22.86" y="93.98"/>
+<instance part="SUPPLY1" gate="+12V" x="182.88" y="147.32"/>
+<instance part="SUPPLY2" gate="GND" x="182.88" y="129.54"/>
+<instance part="C1" gate="G$1" x="190.5" y="139.7"/>
+<instance part="SUPPLY3" gate="+12V" x="190.5" y="157.48" rot="R90"/>
+<instance part="D1" gate="1" x="198.12" y="157.48"/>
 <instance part="SUPPLY6" gate="GND" x="68.58" y="83.82"/>
 <instance part="C2" gate="G$1" x="55.88" y="96.52"/>
@@
 <instance part="SUPPLY13" gate="GND" x="139.7" y="88.9"/>
 <instance part="JP4" gate="A" x="121.92" y="121.92"/>
-<instance part="JP3" gate="A" x="2.54" y="50.8" rot="R180"/>
+<instance part="JP3" gate="A" x="177.8" y="114.3" rot="R180"/>
 <instance part="JP5" gate="A" x="111.76" y="83.82" rot="R180"/>
 <instance part="X1" gate="-1" x="114.3" y="53.34" rot="R180"/>
@@
 <instance part="X2" gate="-2" x="114.3" y="40.64" rot="R180"/>
 <instance part="U$1" gate="G$1" x="0" y="0"/>
+<instance part="X3" gate="-1" x="172.72" y="139.7"/>
+<instance part="X3" gate="-2" x="172.72" y="137.16"/>
 </instances>
 <busses>
@@
 <net name="+12V" class="0">
 <segment>
-<pinref part="J1" gate="G$1" pin="2"/>
 <pinref part="SUPPLY1" gate="+12V" pin="+12V"/>
-<wire x1="2.54" y1="76.2" x2="7.62" y2="76.2" width="0.1524" layer="91"/>
-<wire x1="7.62" y1="76.2" x2="7.62" y2="81.28" width="0.1524" layer="91"/>
-<wire x1="7.62" y1="76.2" x2="10.16" y2="76.2" width="0.1524" layer="91"/>
-<wire x1="10.16" y1="76.2" x2="10.16" y2="78.74" width="0.1524" layer="91"/>
-<junction x="7.62" y="76.2"/>
+<wire x1="177.8" y1="139.7" x2="182.88" y2="139.7" width="0.1524" layer="91"/>
+<wire x1="182.88" y1="139.7" x2="182.88" y2="144.78" width="0.1524" layer="91"/>
+<wire x1="182.88" y1="139.7" x2="185.42" y2="139.7" width="0.1524" layer="91"/>
+<wire x1="185.42" y1="139.7" x2="185.42" y2="142.24" width="0.1524" layer="91"/>
+<junction x="182.88" y="139.7"/>
 <pinref part="C1" gate="G$1" pin="1"/>
-<wire x1="10.16" y1="78.74" x2="15.24" y2="78.74" width="0.1524" layer="91"/>
+<wire x1="185.42" y1="142.24" x2="190.5" y2="142.24" width="0.1524" layer="91"/>
+<pinref part="X3" gate="-1" pin="KL"/>
 </segment>
 <segment>
 <pinref part="SUPPLY3" gate="+12V" pin="+12V"/>
 <pinref part="D1" gate="1" pin="A"/>
-<wire x1="17.78" y1="93.98" x2="20.32" y2="93.98" width="0.1524" layer="91"/>
-<junction x="20.32" y="93.98"/>
-<junction x="17.78" y="93.98"/>
+<wire x1="193.04" y1="157.48" x2="195.58" y2="157.48" width="0.1524" layer="91"/>
+<junction x="195.58" y="157.48"/>
+<junction x="193.04" y="157.48"/>
 </segment>
 </net>
@@
 <segment>
 <pinref part="SUPPLY2" gate="GND" pin="GND"/>
-<wire x1="7.62" y1="68.58" x2="7.62" y2="73.66" width="0.1524" layer="91"/>
-<pinref part="J1" gate="G$1" pin="1"/>
-<wire x1="7.62" y1="73.66" x2="2.54" y2="73.66" width="0.1524" layer="91"/>
-<wire x1="7.62" y1="73.66" x2="10.16" y2="73.66" width="0.1524" layer="91"/>
-<wire x1="10.16" y1="73.66" x2="10.16" y2="71.12" width="0.1524" layer="91"/>
-<junction x="7.62" y="73.66"/>
+<wire x1="182.88" y1="132.08" x2="182.88" y2="137.16" width="0.1524" layer="91"/>
+<wire x1="182.88" y1="137.16" x2="177.8" y2="137.16" width="0.1524" layer="91"/>
+<wire x1="182.88" y1="137.16" x2="185.42" y2="137.16" width="0.1524" layer="91"/>
+<wire x1="185.42" y1="137.16" x2="185.42" y2="134.62" width="0.1524" layer="91"/>
+<junction x="182.88" y="137.16"/>
 <pinref part="C1" gate="G$1" pin="2"/>
-<wire x1="10.16" y1="71.12" x2="15.24" y2="71.12" width="0.1524" layer="91"/>
+<wire x1="185.42" y1="134.62" x2="190.5" y2="134.62" width="0.1524" layer="91"/>
+<pinref part="X3" gate="-2" pin="KL"/>
 </segment>
 <segment>
@@
 <segment>
 <pinref part="JP3" gate="A" pin="2"/>
-<wire x1="5.08" y1="50.8" x2="12.7" y2="50.8" width="0.1524" layer="91"/>
-<label x="12.7" y="50.8" size="1.27" layer="95" xref="yes"/>
+<wire x1="180.34" y1="114.3" x2="187.96" y2="114.3" width="0.1524" layer="91"/>
+<label x="187.96" y="114.3" size="1.27" layer="95" xref="yes"/>
 </segment>
 </net>
@@
 <segment>
 <pinref part="JP3" gate="A" pin="3"/>
-<wire x1="5.08" y1="53.34" x2="12.7" y2="53.34" width="0.1524" layer="91"/>
-<label x="12.7" y="53.34" size="1.27" layer="95" xref="yes"/>
+<wire x1="180.34" y1="116.84" x2="187.96" y2="116.84" width="0.1524" layer="91"/>
+<label x="187.96" y="116.84" size="1.27" layer="95" xref="yes"/>
 </segment>
 </net>
@@
 <segment>
 <pinref part="JP3" gate="A" pin="1"/>
-<wire x1="5.08" y1="48.26" x2="12.7" y2="48.26" width="0.1524" layer="91"/>
-<label x="12.7" y="48.26" size="1.27" layer="95" xref="yes"/>
+<wire x1="180.34" y1="111.76" x2="187.96" y2="111.76" width="0.1524" layer="91"/>
+<label x="187.96" y="111.76" size="1.27" layer="95" xref="yes"/>
 </segment>
 </net>
@@
 <segment>
 <pinref part="D1" gate="1" pin="C"/>
-<wire x1="25.4" y1="93.98" x2="30.48" y2="93.98" width="0.1524" layer="91"/>
-<label x="30.48" y="93.98" size="1.778" layer="95" xref="yes"/>
-<wire x1="25.4" y1="93.98" x2="30.48" y2="93.98" width="0.1524" layer="91"/>
-<label x="30.48" y="93.98" size="1.778" layer="95" xref="yes"/>
-<label x="30.48" y="93.98" size="1.778" layer="95" xref="yes"/>
-<label x="30.48" y="93.98" size="1.778" layer="95" xref="yes"/>
-<junction x="25.4" y="93.98"/>
-<junction x="30.48" y="93.98"/>
-</segment>
-<segment>
+<label x="205.74" y="157.48" size="1.778" layer="95" xref="yes"/>
+<wire x1="200.66" y1="157.48" x2="205.74" y2="157.48" width="0.1524" layer="91"/>
+<label x="205.74" y="157.48" size="1.778" layer="95" xref="yes"/>
+<label x="205.74" y="157.48" size="1.778" layer="95" xref="yes"/>
+<label x="205.74" y="157.48" size="1.778" layer="95" xref="yes"/>
+<junction x="200.66" y="157.48"/>
+<junction x="205.74" y="157.48"/>
+</segment>
+<segment>
